File: Docs/Documents & Advanced/PCB/V3.3/einkPDA_keyboard/einkPDA_keyboard.kicad_pcb (KiCad board)
At the start: 4 copper layers, 95 x 55.5 mm, 126 parts, among them J1 USB_C_Receptacle_USB2.0_16P, J2 Conn_01x12_Pin, J3 Conn_01x26_Pin, J4 Micro_SD_Card, J5 Conn_01x12_Pin, Q1 MMBT3904, SW36 YTS-C017-2B, SW4 SW_DIP_x02, SW43 EVQPUL02K, U1 ESP32-S3-WROOM-1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

Commit message: WIP PCB updates
Routing:
- net SPI_SCK: track 87.9 -> 89.8 mm
