File: Docs/Documents & Advanced/PCB/V3.3/einkPDA_keyboard/einkPDA_keyboard.kicad_sch (KiCad schematic)
At the start: 140 parts, among them J1 USB_C_Receptacle_USB2.0_16P, J2 Conn_01x12_Pin, J3 Conn_01x26_Pin, J4 Micro_SD_Card, J5 Conn_01x12_Pin, Q1 MMBT3904, SW36 YTS-C017-2B, SW4 SW_DIP_x02, SW41 YTS-C017-2B, U1 ESP32-S3-WROOM-1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

Commit message: PCB updates
Parts:
- U1: value ESP32-S3-WROOM-1 -> ESP32-S3-WROOM-1-N16R2
- U8: LCSC Part # C2681320 -> C2680344
Changed lines of the file:
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@@
 			)
 		)
-		(property "LCSC Part #" "C2681320"
+		(property "LCSC Part #" "C2680344"
 			(at 157.48 267.97 0)
 			(effects
@@
 			)
 		)
-		(property "Value" "ESP32-S3-WROOM-1"
+		(property "Value" "ESP32-S3-WROOM-1-N16R2"
 			(at 106.3341 21.59 0)
 			(effects
